File: design_files/AST1029.sch (EAGLE design)
At the start: 3 parts, among them J1 SM05B, SW1 PCM12SMTR

Commit message: updates:
Parts:
- J1: device tinycircuits:AS-ITM-00340 -> tinycircuits:AS-ITM-00340EDGE
Other:
- note added: "Hand Populated: -"
- note added: "Hand Soldered: -"
- note added: "Non Populated: -"
- note added: "Notes: -"
- note added: "Variant: Standard - R"
- note added: "Wireling Small Switch"
- note removed: "Holes need to be moved away from silkscreen"
- note removed: "NOTES:"
